Commit message: modify joint axis direction

File: urdf/p73_walker.urdf (robot description, URDF)
Before this commit: robot p73_walker, 14 links, 13 joints
Links:
- link L_AnkleRoll_Link: geometry collision mesh filename=../meshes/L_AnkleRoll_Link.stl scale=0.001 0.001 0.001; visual mesh filename=../meshes/L_AnkleRoll_Link.stl scale=0.001 0.001 0.001
- link L_Foot_Link: geometry collision mesh filename=../meshes/L_Foot_Link.stl scale=0.001 0.001 0.001; visual mesh filename=../meshes/L_Foot_Link.stl scale=0.001 0.001 0.001
- link L_HipPitch_Link: geometry collision mesh filename=../meshes/L_HipPitch_Link.stl scale=0.001 0.001 0.001; visual mesh filename=../meshes/L_HipPitch_Link.stl scale=0.001 0.001 0.001
- link L_HipRoll_Link: geometry collision mesh filename=../meshes/L_HipRoll_Link.stl scale=0.001 0.001 0.001; visual mesh filename=../meshes/L_HipRoll_Link.stl scale=0.001 0.001 0.001
- link L_Knee_Link: geometry collision mesh filename=../meshes/L_Knee_Link.stl scale=0.001 0.001 0.001; visual mesh filename=../meshes/L_Knee_Link.stl scale=0.001 0.001 0.001
- link L_Thigh_Link: geometry collision mesh filename=../meshes/L_Thigh_Link.stl scale=0.001 0.001 0.001; visual mesh filename=../meshes/L_Thigh_Link.stl scale=0.001 0.001 0.001
- link R_AnkleRoll_Link: geometry collision mesh filename=../meshes/R_AnkleRoll_Link.stl scale=0.001 0.001 0.001; visual mesh filename=../meshes/R_AnkleRoll_Link.stl scale=0.001 0.001 0.001
- link R_Foot_Link: geometry collision mesh filename=../meshes/R_Foot_Link.stl scale=0.001 0.001 0.001; visual mesh filename=../meshes/R_Foot_Link.stl scale=0.001 0.001 0.001
- link R_HipPitch_Link: geometry collision mesh filename=../meshes/R_HipPitch_Link.stl scale=0.001 0.001 0.001; visual mesh filename=../meshes/R_HipPitch_Link.stl scale=0.001 0.001 0.001
- link R_HipRoll_Link: geometry collision mesh filename=../meshes/R_HipRoll_Link.stl scale=0.001 0.001 0.001; visual mesh filename=../meshes/R_HipRoll_Link.stl scale=0.001 0.001 0.001
- link R_Knee_Link: geometry collision mesh filename=../meshes/R_Knee_Link.stl scale=0.001 0.001 0.001; visual mesh filename=../meshes/R_Knee_Link.stl scale=0.001 0.001 0.001
- link R_Thigh_Link: geometry collision mesh filename=../meshes/R_Thigh_Link.stl scale=0.001 0.001 0.001; visual mesh filename=../meshes/R_Thigh_Link.stl scale=0.001 0.001 0.001
- link WaistYaw_Link: geometry collision mesh filename=../meshes/WaistYaw_Link.stl scale=0.001 0.001 0.001; visual mesh filename=../meshes/WaistYaw_Link.stl scale=0.001 0.001 0.001
- link base_link: geometry collision mesh filename=../meshes/base_link.stl scale=0.001 0.001 0.001; visual mesh filename=../meshes/base_link.stl scale=0.001 0.001 0.001
Joints:
- joint L_AnklePitch_Joint: axis 0.0 -1.0 -0.0 -> 0.0 1.0 -0.0; limit lower=-0.7 upper=1.05 effort=95 velocity=10 -> lower=-1.05 upper=0.7 effort=95 velocity=10
- joint L_HipPitch_Joint: axis -0.0 1.0 -0.0 -> -0.0 -1.0 -0.0; limit lower=-2.09 upper=1.57 effort=220.0 velocity=10 -> lower=-1.57 upper=2.09 effort=220.0 velocity=10
- joint L_HipRoll_Joint: axis 1.0 -0.0 0.0 -> -1.0 0.0 0.0; limit lower=-0.58 upper=0.3 effort=352.0 velocity=10 -> lower=-0.3 upper=0.58 effort=352.0 velocity=10
- joint L_Knee_Joint: axis 0.0 -1.0 -0.0 -> 0.0 1.0 -0.0; limit lower=-2.56 upper=0 effort=95 velocity=10 -> lower=0 upper=2.56 effort=95 velocity=10
- joint R_AnklePitch_Joint: axis 0.0 1.0 -0.0 -> 0.0 -1.0 -0.0; limit lower=-1.05 upper=0.7 effort=95 velocity=10 -> lower=-0.7 upper=1.05 effort=95 velocity=10
- joint R_HipPitch_Joint: axis -0.0 -1.0 -0.0 -> -0.0 1.0 -0.0; limit lower=-1.57 upper=2.09 effort=220.0 velocity=10 -> lower=-2.09 upper=1.57 effort=220.0 velocity=10

Commit message: add collision mesh

File: urdf/p73_walker.urdf (robot description, URDF)
Before this commit: robot p73_walker, 14 links, 13 joints
Links:
- link L_Foot_Link: geometry collision box size=0.06 0.1 0.02; collision box size=0.2 0.1 0.02
- link L_HipPitch_Link: geometry collision box size=0.2 0.11 0.26; visual mesh filename=../meshes/L_HipPitch_Link.stl scale=0.001 0.001 0.001
- link L_Knee_Link: geometry collision box size=0.09 0.08 0.16; collision box size=0.12 0.12 0.24
- link L_Thigh_Link: geometry collision box size=0.2 0.14 0.16; visual mesh filename=../meshes/L_Thigh_Link.stl scale=0.001 0.001 0.001
- link R_Foot_Link: geometry collision box size=0.06 0.1 0.02; collision box size=0.2 0.1 0.02
- link R_HipPitch_Link: geometry collision box size=0.2 0.11 0.26; visual mesh filename=../meshes/R_HipPitch_Link.stl scale=0.001 0.001 0.001
- link R_Knee_Link: geometry collision box size=0.09 0.08 0.16; collision box size=0.12 0.12 0.24
- link R_Thigh_Link: geometry collision box size=0.2 0.14 0.16; visual mesh filename=../meshes/R_Thigh_Link.stl scale=0.001 0.001 0.001
- link WaistYaw_Link: geometry collision box size=0.26 0.3 0.4; collision cylinder length=0.04 radius=0.065
- link base_link: geometry collision cylinder length=0.21 radius=0.065; visual mesh filename=../meshes/base_link.stl scale=0.001 0.001 0.001

Commit message: modify hip roll directions

File: urdf/p73_walker.urdf (robot description, URDF)
Before this commit: robot p73_walker, 14 links, 13 joints
Joints:
- joint L_HipRoll_Joint: axis -1.0 0.0 0.0 -> 1.0 0.0 0.0; limit lower=-0.3 upper=0.58 effort=352.0 velocity=10 -> lower=-0.58 upper=0.3 effort=352.0 velocity=10
- joint R_HipRoll_Joint: axis 1.0 -0.0 0.0 -> -1.0 0.0 0.0; limit lower=-0.3 upper=0.58 effort=352.0 velocity=10 -> lower=-0.58 upper=0.3 effort=352.0 velocity=10

Commit message: urdf,xml - modify torque limit

File: urdf/p73_walker.urdf (robot description, URDF)
Before this commit: robot p73_walker, 14 links, 13 joints
Joints:
- joint L_HipYaw_Joint: limit lower=-0.78 upper=0.78 effort=220.0 velocity=10 -> lower=-0.78 upper=0.78 effort=95.0 velocity=10
- joint L_Knee_Joint: limit lower=0 upper=2.56 effort=95 velocity=10 -> lower=0 upper=2.56 effort=220 velocity=10
- joint R_HipYaw_Joint: limit lower=-0.78 upper=0.78 effort=220.0 velocity=10 -> lower=-0.78 upper=0.78 effort=95.0 velocity=10
- joint R_Knee_Joint: limit lower=-2.56 upper=0 effort=95 velocity=10 -> lower=-2.56 upper=0 effort=220 velocity=10

Commit message: urdf - delete ankle collision

File: urdf/p73_walker.urdf (robot description, URDF)
Before this commit: robot p73_walker, 14 links, 13 joints
Links:
- link L_AnkleRoll_Link: geometry visual mesh filename=../meshes/L_AnkleRoll_Link.stl scale=0.001 0.001 0.001
- link R_AnkleRoll_Link: geometry visual mesh filename=../meshes/R_AnkleRoll_Link.stl scale=0.001 0.001 0.001
